File: Mixer Board/TS3A5017-Mixer/_autosave-TS3A5017-Mixer.kicad_sch (KiCad schematic)
At the start: 10 parts, among them J1 RF-In, J2 CLK0, J3 CLK1, J4 Conn_01x06, U1 TS3A5017RGY

Commit message: Continued work and first iteration
Parts:
- J4: footprint (none) -> Connector_PinHeader_2.54mm:PinHeader_1x06_P2.54mm_Vertical
Changed lines of the file:
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@@
 			)
 		)
-		(property "Footprint" ""
+		(property "Footprint" "Connector_PinHeader_2.54mm:PinHeader_1x06_P2.54mm_Vertical"
 			(at 189.23 97.79 0)
 			(effects
