File: Mixer Board/TS3A5017-Mixer/TS3A5017-Mixer.kicad_pcb (KiCad board)
At the start: 2 copper layers, 6 parts, among them J1 Conn_Coaxial_Small, J2 Conn_Coaxial_Small, J3 Conn_Coaxial_Small, U1 TS3A5017RGY, U2 LMP7715MF

Commit message: Continued work and first iteration
Parts:
- removed U2: LMP7715MF, Package_TO_SOT_SMD:SOT-23-5
- added C2: .1uf, Capacitor_SMD:C_1206_3216Metric, F.Cu at (144.9, 99.8)
- added C3: .1uf, Capacitor_SMD:C_1206_3216Metric, F.Cu at (141.2, 99.8)
- added C4: .1uf, Capacitor_SMD:C_1206_3216Metric, F.Cu at (148.5, 99.9)
- added C5: .1uf, Capacitor_SMD:C_1206_3216Metric, F.Cu at (152.1, 99.9)
- added J4: Conn_01x06, Connector_PinHeader_2.54mm:PinHeader_1x06_P2.54mm_Vertical, F.Cu at (140.2, 107.2)
- C1: footprint Capacitor_SMD:C_1206_3216Metric -> Capacitor_SMD:C_0603_1608Metric
- J1: value Conn_Coaxial_Small -> RF-In; footprint Connector_Coaxial:SMA_Amphenol_901-143_Horizontal -> Connector_Amphenol:AMPHENOL_901-143-6RFX
- J2: value Conn_Coaxial_Small -> CLK0; footprint Connector_Coaxial:SMA_Amphenol_901-143_Horizontal -> Connector_Amphenol:AMPHENOL_901-143-6RFX
- J3: value Conn_Coaxial_Small -> CLK1; footprint Connector_Coaxial:SMA_Amphenol_901-143_Horizontal -> Connector_Amphenol:AMPHENOL_901-143-6RFX
- moved J3 19.1 mm to (133.3, 89.9), turned to -90 degrees
- moved U1 18.1 mm to (146.8, 87.9), turned to 180 degrees
- moved J2 16.8 mm to (159.5, 89.9), turned to 90 degrees
- moved J1 16.6 mm to (146.6, 79.2), turned to 180 degrees
- moved C1 10.7 mm to (146.8, 91.4)
Connections:
- net Net-(U1-V+) renamed /3.3V
Routing:
- net Net-(J4-Pin_2): track 0.00 -> 53.5 mm
- net Net-(J4-Pin_3): track 0.00 -> 51.6 mm, vias 0 -> 1
- net Net-(J4-Pin_4): track 0.00 -> 47.3 mm, vias 0 -> 1
- net Net-(J4-Pin_5): track 0.00 -> 47.1 mm, vias 0 -> 1
- net /3.3V: track 0.00 -> 21.7 mm, vias 0 -> 1
- net RF-In: track 0.00 -> 21.5 mm
- net CLK1: track 0.00 -> 12.2 mm, vias 0 -> 1
- net CLK0: track 0.00 -> 11.3 mm, vias 0 -> 1
- net GND: track 0.00 -> 10.4 mm, vias 0 -> 8
- added copper zone on B.Cu, net GND
Other:
- board outline added: 37.8 x 37.1 mm

Commit message: Finish first iteration, generate manufacturing files
Routing:
- net GND: track 10.4 -> 21.7 mm
Other:
- board size 37.8 x 37.1 mm -> 37.8 x 42.9 mm
- board text added: "3.3V"
- board text added: "GND"
- board text added: "I_Neg"
- board text added: "I_Pos"
- board text added: "Q_Neg"
- board text added: "Q_Pos"
Changed lines of the file:
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@@
 			(layer "F.Mask"
 				(type "Top Solder Mask")
-				(color "Black")
 				(thickness 0.01)
 			)
@@
 			(outputformat 1)
 			(mirror no)
-			(drillshape 1)
+			(drillshape 0)
 			(scaleselection 1)
-			(outputdirectory "")
+			(outputdirectory "Manufacture/")
 		)
 	)
@@
 		)
 		(property "Value" ".1uf"
-			(at 0 1.43 360)
+			(at 0 1.43 0)
 			(layer "F.Fab")
+			(hide yes)
 			(effects
 				(font
@@
 		)
 		(fp_text user "${REFERENCE}"
-			(at 0 0 360)
+			(at 0.013 1.016 360)
 			(layer "F.Fab")
 			(effects
@@
 			(at 0.445 -5.889 90)
 			(layer "F.SilkS")
+			(hide yes)
 			(effects
 				(font
@@
 		)
 		(property "Value" "CLK1"
-			(at 14.669 13.111 90)
-			(layer "F.Fab")
+			(at -5.842 0.762 180)
+			(layer "F.SilkS")
 			(effects
 				(font
@@
 			)
 		)
-		(property "Footprint" "Connector_Coaxial:SMA_Amphenol_901-143_Horizontal"
+		(property "Footprint" "Connector_Amphenol:AMPHENOL_901-143-6RFX"
 			(at 0 0 -90)
 			(unlocked yes)
@@
 			)
 		)
+		(property ki_fp_filters "*BNC* *SMA* *SMB* *SMC* *Cinch* *LEMO* *UMRF* *MCX* *U.FL*")
+		(sheetname "Root")
+		(sheetfile "TS3A5017-Mixer.kicad_sch")
 		(attr through_hole)
 		(fp_line
@@
 			(solder_mask_margin 0.102)
 		)
+		(model "${KIPRJMOD}/SMA Connector/901-143-6RFX.step"
+			(offset
+				(xyz 0 0 0)
+			)
+			(scale
+				(xyz 1 1 1)
+			)
+			(rotate
+				(xyz -90 0 0)
+			)
+		)
 	)
 	(footprint "Connector_PinHeader_2.54mm:PinHeader_1x06_P2.54mm_Vertical"
@@
 			(at 0 15.03 270)
 			(layer "F.Fab")
+			(hide yes)
 			(effects
 				(font
@@
 		(at 146.558 79.248 180)
 		(property "Reference" "J1"
-			(at 0.445 -5.889 180)
+			(at 5.334 -0.508 180)
 			(layer "F.SilkS")
+			(hide yes)
 			(effects
 				(font
@@
 		)
 		(property "Value" "RF-In"
-			(at 14.669 13.111 180)
-			(layer "F.Fab")
+			(at 8.128 3.048 180)
+			(layer "F.SilkS")
 			(effects
 				(font
@@
 			)
 		)
-		(property "Footprint" "Connector_Coaxial:SMA_Amphenol_901-143_Horizontal"
+		(property "Footprint" "Connector_Amphenol:AMPHENOL_901-143-6RFX"
 			(at 0 0 180)
 			(unlocked yes)
@@
 			)
 		)
+		(property ki_fp_filters "*BNC* *SMA* *SMB* *SMC* *Cinch* *LEMO* *UMRF* *MCX* *U.FL*")
+		(sheetname "Root")
+		(sheetfile "TS3A5017-Mixer.kicad_sch")
 		(attr through_hole)
 		(fp_line
@@
 			(solder_mask_margin 0.102)
 		)
+		(model "${KIPRJMOD}/SMA Connector/901-143-6RFX.step"
+			(offset
+				(xyz 0 0 0)
+			)
+			(scale
+				(xyz 1 1 1)
+			)
+			(rotate
+				(xyz -90 0 0)
+			)
+		)
 	)
 	(footprint "Connector_Amphenol:AMPHENOL_901-143-6RFX"
@@
 			(at 0.445 -5.889 270)
 			(layer "F.SilkS")
+			(hide yes)
 			(effects
 				(font
@@
 		)
 		(property "Value" "CLK0"
-			(at 14.669 13.111 270)
-			(layer "F.Fab")
+			(at 5.334 0.254 0)
+			(layer "F.SilkS")
 			(effects
 				(font
@@
 			)
 		)
-		(property "Footprint" "Connector_Coaxial:SMA_Amphenol_901-143_Horizontal"
+		(property "Footprint" "Connector_Amphenol:AMPHENOL_901-143-6RFX"
 			(at 0 0 90)
 			(unlocked yes)
@@
 			)
 		)
+		(property ki_fp_filters "*BNC* *SMA* *SMB* *SMC* *Cinch* *LEMO* *UMRF* *MCX* *U.FL*")
+		(sheetname "Root")
+		(sheetfile "TS3A5017-Mixer.kicad_sch")
 		(attr through_hole)
 		(fp_line
@@
 			(solder_mask_margin 0.102)
 		)
+		(model "${KIPRJMOD}/SMA Connector/901-143-6RFX.step"
+			(offset
+				(xyz 0 0 0)
+			)
+			(scale
+				(xyz 1 1 1)
+			)
+			(rotate
+				(xyz -90 0 0)
+			)
+		)
 	)
 	(footprint "Capacitor_SMD:C_1206_3216Metric"
@@
 	(gr_rect
 		(start 127.254 73.66)
-		(end 165.1 110.744)
+		(end 165.1 116.586)
 		(stroke
 			(width 0.05)
@@
 		(layer "Edge.Cuts")
 	)
+	(gr_text "GND"
+		(at 153.924 114.046 90)
+		(layer "F.SilkS" knockout)
+		(effects
+			(font
+				(size 1.5 1.5)
+				(thickness 0.3)
+				(bold yes)
+			)
+			(justify left bottom)
+		)
+	)
+	(gr_text "Q_Neg"
+		(at 148.475053 116.166525 90)
+		(layer "F.SilkS" knockout)
+		(effects
+			(font
+				(size 1.5 1.5)
+				(thickness 0.3)
+				(bold yes)
+			)
+			(justify left bottom)
+		)
+	)
+	(gr_text "Q_Pos"
+		(at 151.13 115.824 90)
+		(layer "F.SilkS")
+		(effects
+			(font
+				(size 1.5 1.5)
+				(thickness 0.3)
+				(bold yes)
+			)
+			(justify left bottom)
+		)
+	)
+	(gr_text "I_Neg"
+		(at 143.51 115.316 90)
+		(layer "F.SilkS" knockout)
+		(effects
+			(font
+				(size 1.5 1.5)
+				(thickness 0.3)
+				(bold yes)
+			)
+			(justify left bottom)
+		)
+	)
+	(gr_text "3.3V"
+		(at 141.224 114.046 90)
+		(layer "F.SilkS")
+		(effects
+			(font
+				(size 1.5 1.5)
+				(thickness 0.3)
+				(bold yes)
+			)
+			(justify left bottom)
+		)
+	)
+	(gr_text "I_Pos"
+		(at 146.05 115.062 90)
+		(layer "F.SilkS")
+		(effects
+			(font
+				(size 1.5 1.5)
+				(thickness 0.3)
+				(bold yes)
+			)
+			(justify left bottom)
+		)
+	)
 	(segment
 		(start 146.037 91.427)
@@
 	)
 	(segment
-		(start 147.537 89.916)
-		(end 147.537 91.403)
+		(start 148.505332 101.346)
+		(end 152.146 101.346)
 		(width 0.2)
 		(layer "F.Cu")
@@
 	)
 	(segment
-		(start 144.305 89.121)
-		(end 143.764 89.662)
+		(start 148.456332 101.297)
+		(end 148.505332 101.346)
 		(width 0.2)
 		(layer "F.Cu")
@@
 	)
 	(segment
-		(start 148.505332 101.346)
-		(end 148.505332 102.446668)
+		(start 147.537 89.916)
+		(end 147.537 91.403)
+		(width 0.2)
+		(layer "F.Cu")
+		(net 2)
+	)
+	(segment
+		(start 144.305 89.121)
+		(end 143.764 89.662)
 		(width 0.2)
 		(layer "F.Cu")
@@
 	)
 	(segment
-		(start 148.505332 102.446668)
-		(end 148.336 102.616)
+		(start 148.505332 101.346)
+		(end 146.812 101.346)
 		(width 0.2)
 		(layer "F.Cu")
@@
 	)
 	(segment
+		(start 141.224 101.297)
+		(end 144.864666 101.297)
+		(width 0.2)
+		(layer "F.Cu")
+		(net 2)
+	)
+	(segment
+		(start 144.864666 101.297)
+		(end 148.456332 101.297)
+		(width 0.2)
+		(layer "F.Cu")
+		(net 2)
+	)
+	(segment
 		(start 147.537 91.403)
 		(end 147.574 91.44)
@@
 	)
 	(via
-		(at 148.336 102.616)
-		(size 0.6)
-		(drill 0.3)
-		(layers "F.Cu" "B.Cu")
-		(net 2)
-	)
-	(via
 		(at 141.224 102.616)
 		(size 0.6)
@@
 		(net 2)
 	)
+	(via
+		(at 146.812 101.346)
+		(size 0.6)
+		(drill 0.3)
+		(layers "F.Cu" "B.Cu")
+		(net 2)
+	)
 	(segment
-		(start 146.037 79.769)
-		(end 146.558 79.248)
+		(start 146.037 85.826)
+		(end 146.037 79.769)
 		(width 0.2)
 		(layer "F.Cu")
@@
 	)
 	(segment
+		(start 146.037 79.769)
+		(end 146.558 79.248)
+		(width 0.2)
+		(layer "F.Cu")
+		(net 3)
+	)
+	(segment
 		(start 151.13 79.248)
 		(end 146.558 79.248)
@@
 	)
 	(segment
-		(start 146.037 85.826)
-		(end 146.037 79.769)
-		(width 0.2)
-		(layer "F.Cu")
-		(net 3)
-	)
-	(segment
 		(start 149.065 89.121)
 		(end 149.86 89.916)
@@
 		(polygon
 			(pts
-				(xy 124.46 70.866) (xy 167.64 70.866) (xy 167.386 111.76) (xy 124.206 111.76)
+				(xy 124.46 70.866) (xy 167.64 70.866) (xy 167.386 117.094) (xy 124.206 117.094)
 			)
 		)
